File: iolink.kicad_sch (KiCad schematic)
At the start: 47 parts, among them IC1 LTC2874IFE#PBF, IC2 AZ1117CH2-5.0TRG1, IC3 M78AR05-0.5, IC4 CH224K, J1 Screw_Terminal_01x04, J2 USB_C_Receptacle_USB2.0, J3 Screw_Terminal_01x05, J4 Screw_Terminal_01x04, J5 Screw_Terminal_01x04, J6 Screw_Terminal_01x04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

Commit message: temp
Parts:
- added C17: 0.1uF, Capacitor_SMD:C_0603_1608Metric, symbol Device:C
- added C18: 4.7uF, Capacitor_SMD:C_0603_1608Metric, symbol Device:C
Connections:
- net +3V3: now also C17.1, C18.1
- net CAN_H: now also J1.4 (Pin_4); no longer J1.3 (Pin_3)
- net CAN_L: now also J1.3 (Pin_3); no longer J1.4 (Pin_4)
- net GND: now also C17.2, C18.2
Other:
- moved on the sheet: C10, C11, C12, C13, C8, C9

Commit message: complete
Parts:
- removed J3: Screw_Terminal_01x05, TerminalBlock_Phoenix:TerminalBlock_Phoenix_MPT-0,5-5-2.54_1x05_P2.54mm_Horizontal, symbol Connector:Screw_Terminal_01x05
- added J8: Screw_Terminal_01x06, TerminalBlock_Phoenix:TerminalBlock_Phoenix_MPT-0,5-6-2.54_1x06_P2.54mm_Horizontal, symbol Connector:Screw_Terminal_01x06
- C14: value C -> 0.1uF
- C5: value 47uF -> 4.7uF
- C7, C9: value 4.7uF -> 0.1uF
- C8: value 0.1uF -> 4.7uF
- SW1: footprint Button_Switch_SMD:SW_SPST_FSMSM -> Button_Switch_THT:SW_PUSH_6mm_H4.3mm
Connections:
- net +5V: now also J8.2 (Pin_2)
- net GND: now also J8.1 (Pin_1)
- net SWCLK: now also J8.4 (Pin_4)
- net SWDIO: now also J8.3 (Pin_3)
- net USART1_RX: now also J8.6 (Pin_6)
- net USART1_TX: now also J8.5 (Pin_5)
